Commit message: updated spray bottle asset and fixed target_dof

File: assets/urdf/objects/spray_bottle/mobility.urdf (robot description, URDF)
Before this commit: robot partnet_367a3f80-12b1-40f7-b343-6392b40a5c7e, 7 links, 6 joints
Links:
- link link_0: geometry collision mesh filename=textured_objs/original-20.obj scale=0.2 0.2 0.2; visual mesh filename=textured_objs/original-20.obj scale=0.2 0.2 0.2
- link link_1: geometry collision mesh filename=textured_objs/original-1.obj scale=0.2 0.2 0.2; collision mesh filename=textured_objs/original-10.obj scale=0.2 0.2 0.2
- link link_2: geometry collision mesh filename=textured_objs/original-16.obj scale=0.2 0.2 0.2; visual mesh filename=textured_objs/original-16.obj scale=0.2 0.2 0.2
- link link_3: geometry collision mesh filename=textured_objs/original-2.obj scale=0.2 0.2 0.2; collision mesh filename=textured_objs/original-3.obj scale=0.2 0.2 0.2
Joints:
- joint joint_0: limit lower=0.0 upper=0.7853981633974483 -> lower=0.0 upper=0.07853981633974483
- joint joint_1: type continuous -> fixed
- joint joint_2: type continuous -> fixed
- joint joint_4: type prismatic -> fixed
- joint joint_5: type prismatic -> fixed
