Commit message: changed size of dispenser, changed hand to floating

File: assets/urdf/kuka_allegro_description/allegro.urdf (robot description, URDF)
Before this commit: robot kuka_allegro, 22 links, 20 joints
Joints:
- joint allegro_mount_joint: type fixed -> floating

File: assets/urdf/objects/dispenser/mobility.urdf (robot description, URDF)
Before this commit: robot partnet_5ca994bd512be485db3bac7ad77ae88e, 4 links, 3 joints
Links:
- link link_0: geometry collision mesh filename=textured_objs/new-0.obj scale=0.1 0.1 0.1; collision mesh filename=textured_objs/new-1.obj scale=0.1 0.1 0.1
- link link_1: geometry collision mesh filename=textured_objs/new-2.obj scale=0.1 0.1 0.1; collision mesh filename=textured_objs/new-4.obj scale=0.1 0.1 0.1

Commit message: Added full articulation of allegro hand (xyz position + orientation)

File: assets/urdf/kuka_allegro_description/allegro.urdf (robot description, URDF)
Before this commit: robot kuka_allegro, 22 links, 21 joints
Joints:
- joint allegro_mount_joint: type floating -> fixed

File: assets/urdf/kuka_allegro_description/allegro_grasp_test.urdf (robot description, URDF)
Before this commit: robot kuka_allegro, 27 links, 26 joints
Links:
- link allegro_mount: geometry collision mesh filename=meshes/mounts/allegro_mount.obj; visual mesh filename=meshes/mounts/allegro_mount.obj
- link index_biotac_tip: geometry collision mesh filename=meshes/biotac/collision/biotac_sensor_tip.obj; visual mesh filename=meshes/biotac/visual/biotac_sensor_tip.obj
- link index_link_0: geometry collision mesh filename=meshes/allegro/primary_base.obj; visual mesh filename=meshes/allegro/primary_base.obj
- link index_link_1: geometry collision mesh filename=meshes/allegro/primary_proximal.obj; visual mesh filename=meshes/allegro/primary_proximal.obj
- link index_link_2: geometry collision mesh filename=meshes/allegro/primary_medial.obj; visual mesh filename=meshes/allegro/primary_medial.obj
- link index_link_3: geometry collision mesh filename=meshes/biotac/collision/biotac_sensor_base.obj; visual mesh filename=meshes/biotac/visual/biotac_sensor_base.obj
- link middle_biotac_tip: geometry collision mesh filename=meshes/biotac/collision/biotac_sensor_tip.obj; visual mesh filename=meshes/biotac/visual/biotac_sensor_tip.obj
- link middle_link_0: geometry collision mesh filename=meshes/allegro/primary_base.obj; visual mesh filename=meshes/allegro/primary_base.obj
- link middle_link_1: geometry collision mesh filename=meshes/allegro/primary_proximal.obj; visual mesh filename=meshes/allegro/primary_proximal.obj
- link middle_link_2: geometry collision mesh filename=meshes/allegro/primary_medial.obj; visual mesh filename=meshes/allegro/primary_medial.obj
- link middle_link_3: geometry collision mesh filename=meshes/biotac/collision/biotac_sensor_base.obj; visual mesh filename=meshes/biotac/visual/biotac_sensor_base.obj
- link palm_link: geometry collision mesh filename=meshes/allegro/base_link.obj; visual mesh filename=meshes/allegro/base_link.obj
- link ring_biotac_tip: geometry collision mesh filename=meshes/biotac/collision/biotac_sensor_tip.obj; visual mesh filename=meshes/biotac/visual/biotac_sensor_tip.obj
- link ring_link_0: geometry collision mesh filename=meshes/allegro/primary_base.obj; visual mesh filename=meshes/allegro/primary_base.obj
- link ring_link_1: geometry collision mesh filename=meshes/allegro/primary_proximal.obj; visual mesh filename=meshes/allegro/primary_proximal.obj
- link ring_link_2: geometry collision mesh filename=meshes/allegro/primary_medial.obj; visual mesh filename=meshes/allegro/primary_medial.obj
- link ring_link_3: geometry collision mesh filename=meshes/biotac/collision/biotac_sensor_base.obj; visual mesh filename=meshes/biotac/visual/biotac_sensor_base.obj
- link thumb_biotac_tip: geometry collision mesh filename=meshes/biotac/collision/biotac_sensor_thumb_tip.obj; visual mesh filename=meshes/biotac/visual/biotac_sensor_thumb_tip.obj
- link thumb_link_0: geometry collision mesh filename=meshes/allegro/thumb_base.obj; visual mesh filename=meshes/allegro/thumb_base.obj
- link thumb_link_1: geometry collision mesh filename=meshes/allegro/thumb_proximal.obj; visual mesh filename=meshes/allegro/thumb_proximal.obj
- link thumb_link_2: geometry collision mesh filename=meshes/allegro/thumb_medial.obj; visual mesh filename=meshes/allegro/thumb_medial.obj
- link thumb_link_3: geometry collision mesh filename=meshes/biotac/collision/biotac_sensor_thumb_base.obj; visual mesh filename=meshes/biotac/visual/biotac_sensor_thumb_base.obj
Joints:
- joint allegro_mount_joint_x: axis 1 0 0 -> (none)
- joint allegro_mount_joint_z: axis 0 1 0 -> 0 0 1
