Commit message: adds obs_dict functionality to articulate tasks
- adds actor_critic_dict network for training multi-task PPO
- adds configs for ArticulateTask with Camera inputs
- cleanup dispenser object
- add tip-over penalty to rewards
- leave allegro_grasp urdf unfixed, and create new one (fixed)
- add schedule to reset position noise for training with curriculum
- set object mass to 1 (much less than previous)

File: assets/urdf/kuka_allegro_description/allegro_grasp.urdf (robot description, URDF)
Before this commit: robot kuka_allegro, 27 links, 26 joints
Joints:
- joint allegro_mount_joint_y: axis 0 1 0 -> 0 0 1

File: assets/urdf/objects/dispenser/mobility.urdf (robot description, URDF)
Before this commit: robot partnet_5ca994bd512be485db3bac7ad77ae88e, 4 links, 3 joints
Joints:
- joint joint_0: origin xyz=0.004069706478648613 0 0.007451467190511252 -> xyz=0.0007326071661966703 0 0.0013411640742919854
