Commit message: fix spray3 object, config, and articulate

File: assets/urdf/objects/spray_bottle3/mobility.urdf (robot description, URDF)
Before this commit: robot partnet_e27e2864f9b54ca5bf9a3f8c45e44354, 5 links, 4 joints
Links:
- link link_0: geometry collision mesh filename=textured_objs/original-5.obj scale=0.2 0.2 0.2; visual mesh filename=textured_objs/original-5.obj scale=0.2 0.2 0.2
- link link_1: geometry collision mesh filename=textured_objs/original-3.obj scale=0.2 0.2 0.2; collision mesh filename=textured_objs/original-4.obj scale=0.2 0.2 0.2
- link link_2: geometry collision mesh filename=textured_objs/original-1.obj scale=0.2 0.2 0.2; visual mesh filename=textured_objs/original-1.obj scale=0.2 0.2 0.2
Joints:
- joint joint_0: origin xyz=0.0244558505733485 0.823748013051608 0.1646802698159997 -> xyz=0.0048911701146697 0.1647496026103216 0.03293605396319994
- joint joint_1: axis 0 1 0 -> (none); type continuous -> fixed
- joint joint_3: axis 0 1 0 -> (none); limit lower=0 upper=0.10000000000000009 -> (none); origin xyz=0.0059191494266517646 0 -0.010204229854504095 -> xyz=0.001183829885330353 0 -0.002040845970900819; type prismatic -> fixed
