Commit message: added joint to allegro urdf and set default pos to open hand

File: assets/urdf/objects/dispenser/mobility.urdf (robot description, URDF)
Before this commit: robot partnet_5ca994bd512be485db3bac7ad77ae88e, 4 links, 3 joints
Links:
- link link_0: geometry collision mesh filename=textured_objs/new-0.obj scale=0.18 0.18 0.18; collision mesh filename=textured_objs/new-1.obj scale=0.18 0.18 0.18
- link link_1: geometry collision mesh filename=textured_objs/new-2.obj scale=0.18 0.18 0.18; collision mesh filename=textured_objs/new-4.obj scale=0.18 0.18 0.18
Joints:
- joint joint_0: axis 0 1 0 -> (none); type continuous -> fixed
- joint joint_2: limit lower=0 upper=0.08400000000000007 -> lower=0 upper=0.015

Commit message: Adds ArticulateTask to tasks
- creates multiple object instances and object types
- issue: fix when multiple objects types and instances are used
  (current indexing doesn't work)
- adds object task rewards for access to hyperparams and reward
  functions from cli

File: assets/urdf/objects/dispenser/mobility.urdf (robot description, URDF)
Before this commit: robot partnet_5ca994bd512be485db3bac7ad77ae88e, 4 links, 3 joints
Joints:
- removed joint joint_1
- removed joint joint_2
- added joint fixed_joint_0: type fixed, parent link_0_helper, child link_0, origin xyz=0.0 0 0.0
- added joint fixed_joint_1: type fixed, parent base, child link_1, origin xyz=0 0 0 rpy=1.570796326794897 0 -1.570796326794897
- joint joint_0: axis (none) -> 0 -1 0; child link_0 -> link_0_helper; limit (none) -> lower=0 upper=0.015; origin xyz=0.0 0 0.0 -> xyz=0.004069706478648613 0 0.007451467190511252; parent link_0_helper -> link_1; type fixed -> prismatic

Commit message: added dispenser config, fix spraybottle5

File: assets/urdf/objects/dispenser/mobility.urdf (robot description, URDF)
Before this commit: robot partnet_5ca994bd512be485db3bac7ad77ae88e, 4 links, 3 joints
Links:
- link link_0: geometry collision mesh filename=textured_objs/original-2.obj scale=0.2 0.2 0.2; collision mesh filename=textured_objs/original-3.obj scale=0.2 0.2 0.2
- link link_1: geometry collision mesh filename=textured_objs/original-1.obj scale=0.2 0.2 0.2; visual mesh filename=textured_objs/original-1.obj scale=0.2 0.2 0.2
Joints:
- joint fixed_joint_0: axis (none) -> 0 1 0
- joint joint_0: limit lower=0 upper=0.015 -> lower=0. upper=0.04; origin xyz=0.0007326071661966703 0 0.0013411640742919854 -> xyz=-0.0017510127982153934 0 -0.00274114442045887

File: assets/urdf/objects/spray_bottle4/mobility.urdf (robot description, URDF)
Before this commit: robot partnet_2a9b20d21e27ab0026cca18be86a1458, 5 links, 4 joints
Links:
- link link_0: geometry collision mesh filename=textured_objs/original-12.obj scale=0.2 0.2 0.2; visual mesh filename=textured_objs/original-12.obj scale=0.2 0.2 0.2
- link link_1: geometry collision mesh filename=textured_objs/original-29.obj scale=0.2 0.2 0.2; collision mesh filename=textured_objs/original-29.obj scale=0.2 0.2 0.2
- link link_2: geometry collision mesh filename=textured_objs/original-8.obj scale=0.2 0.2 0.2; visual mesh filename=textured_objs/original-11.obj scale=0.2 0.2 0.2
Joints:
- joint joint_0: origin xyz=0.05938179134939801 0.8545218342536304 0.08651277610414826 -> xyz=0.011876358269879602 0.17090436685072608 0.017302555220829652
- joint joint_3: axis 0 1 0 -> (none); limit lower=0 upper=0.12 effort=100.0 velocity=1 -> (none); origin xyz=0.0008504999999999971 0 -0.004366499999999999 -> xyz=0.00017009999999999943 0 -0.0008732999999999998; type prismatic -> fixed

File: assets/urdf/objects/spray_bottle5/mobility.urdf (robot description, URDF)
Before this commit: robot partnet_5ca994bd512be485db3bac7ad77ae88e, 4 links, 3 joints
Links:
- removed link link_0_helper
- added link link_2; collision mesh filename=textured_objs/original-10.obj scale=0.2 0.2 0.2; collision mesh filename=textured_objs/original-11.obj scale=0.2 0.2 0.2
- added link link_2_helper
- link link_0: geometry collision mesh filename=textured_objs/original-6.obj scale=0.2 0.2 0.2; collision mesh filename=textured_objs/original-9.obj scale=0.2 0.2 0.2
- link link_1: geometry collision mesh filename=textured_objs/original-1.obj scale=0.2 0.2 0.2; visual mesh filename=textured_objs/original-1.obj scale=0.2 0.2 0.2
Joints:
- added joint joint_3: type fixed, parent link_1, child link_2_helper, origin xyz=-0.0010098984132660596 0 -0.0018723025097779692, axis 0 1 0, limit lower=-0.04800000000000004 upper=-0.008000000000000007
- joint joint_0: axis 0 1 0 -> 1 0 0; limit (none) -> lower=0.0 upper=0.36442474781641604; origin xyz=0.0 0 0.0 -> xyz=0.014137898413266086 0.14960500398709136 0.044993421453171556; parent link_0_helper -> link_2; type fixed -> revolute
- joint joint_2: axis 0 -1 0 -> 0 1 0; child link_0_helper -> link_2; limit lower=-0.1 upper=0.1 -> (none); origin xyz=-0.008755063991076967 0 -0.01370572210229435 -> xyz=0.0 0 0.0; parent link_1 -> link_2_helper; type prismatic -> fixed
