Commit message: added dof_scaled keys to base config
- added damping and stiffness to each object
- set 0 stiffness for scissors

File: assets/urdf/objects/spray_bottle2/mobility.urdf (robot description, URDF)
Before this commit: robot partnet_a7732257-2737-4c45-aaa2-b2c8a65c5fe8, 5 links, 4 joints
Joints:
- joint joint_0: limit lower=-0.0 upper=0.3490658503988659 -> lower=-0.0 upper=0.085

File: assets/urdf/objects/spray_bottle3/mobility.urdf (robot description, URDF)
Before this commit: robot partnet_e27e2864f9b54ca5bf9a3f8c45e44354, 5 links, 4 joints
Joints:
- joint joint_0: limit lower=-0.0 upper=1.0471975511965976 -> lower=0.0 upper=1.0471975511965976
